File: pcb/autotome.kicad_sch (KiCad schematic)
At the start: 62 parts, among them SW1 SW_PUSH, SW10 SW_PUSH, SW11 SW_PUSH, SW12 SW_PUSH, SW13 SW_PUSH, SW14 SW_PUSH, SW15 SW_PUSH, SW16 SW_PUSH, SW17 SW_PUSH, SW18 SW_PUSH, SW19 SW_PUSH, SW2 SW_PUSH, SW20 SW_PUSH, SW21 SW_PUSH, SW22 SW_PUSH, SW23 SW_PUSH, SW24 SW_PUSH, SW25 RotaryEncoder_Switch, SW26 SW_PUSH, SW27 SW_PUSH, SW28 SW_PUSH, SW29 SW_PUSH, SW3 SW_PUSH, SW30 SW_PUSH, SW31 SW_SPDT, SW4 SW_PUSH, SW5 SW_PUSH, SW6 SW_PUSH, SW7 SW_PUSH, SW8 SW_PUSH, SW9 SW_PUSH, U1 ProMicro

Commit message: fix schematic - connect enc switch diode to row
Connections:
- net col 6: now also SW25.S1; no longer D25.1 (K)
- net row 3: now also D25.1 (K); no longer SW25.S2
- net at D25.2 (A): now also SW25.S2; no longer SW25.S1
Other:
- moved on the sheet: D25, SW25
Changed lines of the file:
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@@
 	)
 	(junction
+		(at 147.32 123.19)
+		(diameter 0)
+		(color 0 0 0 0)
+	)
+	(junction
 		(at 104.14 113.03)
 		(diameter 0)
@@
 	)
 	(junction
-		(at 127 123.19)
-		(diameter 0)
-		(color 0 0 0 0)
-	)
-	(junction
 		(at 71.12 105.41)
 		(diameter 0)
@@
 	(wire
 		(pts
-			(xy 127 123.19) (xy 143.51 123.19)
-		)
-		(stroke
-			(width 0)
-			(type default)
-		)
-	)
-	(wire
-		(pts
 			(xy 106.68 85.09) (xy 106.68 95.25)
 		)
@@
 	(wire
 		(pts
-			(xy 121.92 123.19) (xy 127 123.19)
+			(xy 121.92 123.19) (xy 147.32 123.19)
 		)
 		(stroke
@@
 	(wire
 		(pts
-			(xy 35.56 85.09) (xy 35.56 95.25)
+			(xy 160.02 115.57) (xy 152.4 115.57)
 		)
 		(stroke
@@
 	(wire
 		(pts
-			(xy 88.9 85.09) (xy 88.9 95.25)
+			(xy 158.75 123.19) (xy 147.32 123.19)
 		)
 		(stroke
@@
 	(wire
 		(pts
-			(xy 35.56 105.41) (xy 35.56 115.57)
+			(xy 35.56 85.09) (xy 35.56 95.25)
 		)
 		(stroke
@@
 	(wire
 		(pts
-			(xy 106.68 95.25) (xy 106.68 105.41)
+			(xy 88.9 85.09) (xy 88.9 95.25)
 		)
 		(stroke
@@
 	(wire
 		(pts
-			(xy 17.78 85.09) (xy 17.78 95.25)
+			(xy 35.56 105.41) (xy 35.56 115.57)
 		)
 		(stroke
@@
 	(wire
 		(pts
-			(xy 127 119.38) (xy 127 123.19)
+			(xy 106.68 95.25) (xy 106.68 105.41)
+		)
+		(stroke
+			(width 0)
+			(type default)
+		)
+	)
+	(wire
+		(pts
+			(xy 17.78 85.09) (xy 17.78 95.25)
 		)
 		(stroke
@@
 	(global_label "row 3"
 		(shape input)
-		(at 127 119.38 0)
+		(at 158.75 123.19 0)
 		(fields_autoplaced yes)
 		(effects
@@
 		)
 		(property "Intersheetrefs" "${INTERSHEET_REFS}"
-			(at 135.428 119.38 0)
+			(at 167.178 123.19 0)
 			(hide yes)
 			(show_name no)
@@
 	(global_label "enc A"
 		(shape input)
-		(at 148.59 107.95 90)
+		(at 152.4 100.33 90)
 		(fields_autoplaced yes)
 		(effects
@@
 		)
 		(property "Intersheetrefs" "${INTERSHEET_REFS}"
-			(at 148.59 99.5824 90)
+			(at 152.4 91.9624 90)
 			(hide yes)
 			(show_name no)
@@
 	(global_label "col 6"
 		(shape input)
-		(at 148.59 130.81 270)
+		(at 160.02 115.57 0)
 		(fields_autoplaced yes)
 		(effects
@@
 				(size 1.27 1.27)
 			)
-			(justify right)
+			(justify left)
 		)
 		(property "Intersheetrefs" "${INTERSHEET_REFS}"
-			(at 148.59 138.8751 90)
+			(at 168.0851 115.57 0)
 			(hide yes)
 			(show_name no)
@@
 					(size 1.27 1.27)
 				)
-				(justify right)
+				(justify left)
 			)
 		)
@@
 	(global_label "B-"
 		(shape input)
-		(at 146.05 107.95 90)
+		(at 149.86 100.33 90)
 		(fields_autoplaced yes)
 		(effects
@@
 		)
 		(property "Intersheetrefs" "${INTERSHEET_REFS}"
-			(at 146.05 102.1224 90)
+			(at 149.86 94.5024 90)
 			(hide yes)
 			(show_name no)
@@
 	(global_label "enc B"
 		(shape input)
-		(at 143.51 107.95 90)
+		(at 147.32 100.33 90)
 		(fields_autoplaced yes)
 		(effects
@@
 		)
 		(property "Intersheetrefs" "${INTERSHEET_REFS}"
-			(at 143.51 99.401 90)
+			(at 147.32 91.781 90)
 			(hide yes)
 			(show_name no)
@@
 	(symbol
 		(lib_id "Device:RotaryEncoder_Switch")
-		(at 146.05 115.57 270)
+		(at 149.86 107.95 270)
 		(unit 1)
 		(body_style 1)
@@
 		(fields_autoplaced yes)
 		(property "Reference" "SW25"
-			(at 152.4 114.2999 90)
+			(at 156.21 106.6799 90)
 			(show_name no)
 			(do_not_autoplace no)
@@
 		)
 		(property "Value" "RotaryEncoder_Switch"
-			(at 152.4 116.8399 90)
+			(at 156.21 109.2199 90)
 			(show_name no)
 			(do_not_autoplace no)
@@
 		)
 		(property "Footprint" "Rotary_Encoder:RotaryEncoder_Alps_EC11E-Switch_Vertical_H20mm"
-			(at 150.114 111.76 0)
+			(at 153.924 104.14 0)
 			(hide yes)
 			(show_name no)
@@
 		)
 		(property "Datasheet" ""
-			(at 152.654 115.57 0)
+			(at 156.464 107.95 0)
 			(hide yes)
 			(show_name no)
@@
 		)
 		(property "Description" "Rotary encoder, dual channel, incremental quadrate outputs, with switch"
-			(at 146.05 115.57 0)
+			(at 149.86 107.95 0)
 			(hide yes)
 			(show_name no)
@@
 	(symbol
 		(lib_id "Diode:1N4148")
-		(at 148.59 127 90)
+		(at 147.32 119.38 90)
 		(unit 1)
 		(body_style 1)
@@
 		(dnp no)
 		(property "Reference" "D25"
-			(at 147.32 127 90)
+			(at 149.606 120.65 90)
 			(show_name no)
 			(do_not_autoplace no)
@@
 		)
 		(property "Value" "1N4148"
-			(at 138.684 128.27 90)
+			(at 137.414 120.65 90)
 			(show_name no)
 			(do_not_autoplace no)
@@
 		)
 		(property "Footprint" "Diode_THT:D_DO-35_SOD27_P7.62mm_Horizontal"
-			(at 148.59 127 0)
+			(at 147.32 119.38 0)
 			(hide yes)
 			(show_name no)
@@
 		)
 		(property "Datasheet" "https://assets.nexperia.com/documents/data-sheet/1N4148_1N4448.pdf"
-			(at 148.59 127 0)
+			(at 147.32 119.38 0)
 			(hide yes)
 			(show_name no)
@@
 		)
 		(property "Description" "100V 0.15A standard switching diode, DO-35"
-			(at 148.59 127 0)
+			(at 147.32 119.38 0)
 			(hide yes)
 			(show_name no)
@@
 		)
 		(property "Sim.Device" "D"
-			(at 148.59 127 0)
+			(at 147.32 119.38 0)
 			(hide yes)
 			(show_name no)
@@
 		)
 		(property "Sim.Pins" "1=K 2=A"
-			(at 148.59 127 0)
+			(at 147.32 119.38 0)
 			(hide yes)
 			(show_name no)

Commit message: remove reset button from schematic
will be wired direcly on top of the controller
Parts:
- removed SW26: SW_PUSH, Button_Switch_THT:SW_PUSH_6mm, symbol kbd:SW_PUSH
Changed lines of the file:
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@@
 		)
 	)
-	(global_label "B-"
-		(shape input)
-		(at 109.22 24.13 0)
-		(fields_autoplaced yes)
-		(effects
-			(font
-				(size 1.27 1.27)
-			)
-			(justify left)
-		)
-		(property "Intersheetrefs" "${INTERSHEET_REFS}"
-			(at 115.0476 24.13 0)
-			(hide yes)
-			(show_name no)
-			(do_not_autoplace no)
-			(effects
-				(font
-					(size 1.27 1.27)
-				)
-				(justify left)
-			)
-		)
-	)
 	(global_label "col 4"
 		(shape input)
@@
 		)
 	)
-	(global_label "RST"
-		(shape input)
-		(at 93.98 24.13 180)
-		(fields_autoplaced yes)
-		(effects
-			(font
-				(size 1.27 1.27)
-			)
-			(justify right)
-		)
-		(property "Intersheetrefs" "${INTERSHEET_REFS}"
-			(at 87.5477 24.13 0)
-			(hide yes)
-			(show_name no)
-			(do_not_autoplace no)
-			(effects
-				(font
-					(size 1.27 1.27)
-				)
-				(justify right)
-			)
-		)
-	)
 	(global_label "row 4"
 		(shape input)
@@
 					(unit 1)
 				)
-			)
-		)
-	)
-	(symbol
-		(lib_id "kbd:SW_PUSH")
-		(at 101.6 24.13 0)
-		(unit 1)
-		(body_style 1)
-		(exclude_from_sim no)
-		(in_bom yes)
-		(on_board yes)
-		(in_pos_files yes)
-		(dnp no)
-		(property "Reference" "SW26"
-			(at 101.6 19.812 0)
-			(show_name no)
-			(do_not_autoplace no)
-			(effects
-				(font
-					(size 1.27 1.27)
-				)
-			)
-		)
-		(property "Value" "SW_PUSH"
-			(at 101.6 26.162 0)
-			(show_name no)
-			(do_not_autoplace no)
-			(effects
-				(font
-					(size 1.27 1.27)
-				)
-			)
-		)
-		(property "Footprint" "Button_Switch_THT:SW_PUSH_6mm"
-			(at 101.6 24.13 0)
-			(hide yes)
-			(show_name no)
-			(do_not_autoplace no)
-			(effects
-				(font
-					(size 1.27 1.27)
-				)
-			)
-		)
-		(property "Datasheet" ""
-			(at 101.6 24.13 0)
-			(show_name no)
-			(do_not_autoplace no)
-			(effects
-				(font
-					(size 1.27 1.27)
-				)
-			)
-		)
-		(property "Description" ""
-			(at 101.6 24.13 0)
-			(hide yes)
-			(show_name no)
-			(do_not_autoplace no)
-			(effects
-				(font
-					(size 1.27 1.27)
-				)
-			)
-		)
-		(pin "1"
-		)
-		(pin "2"
-		)
-		(instances
-			(project "autotome"
-				(path "/7a8f7727-35b5-4a31-8719-22ef542e3f8e"
-					(reference "SW26")
-					(unit 1)
-				)

Commit message: add rotary encoder 3d model and custom library
Parts:
- SW25: footprint Rotary_Encoder:RotaryEncoder_Alps_EC11E-Switch_Vertical_H20mm -> my_library:RotaryEncoder_Alps_EC11E-Switch_Vertical_H20mm
Changed lines of the file:
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@@
 			)
 		)
-		(property "Footprint" "Rotary_Encoder:RotaryEncoder_Alps_EC11E-Switch_Vertical_H20mm"
+		(property "Footprint" "my_library:RotaryEncoder_Alps_EC11E-Switch_Vertical_H20mm"
 			(at 153.924 104.14 0)
 			(hide yes)

Commit message: add nice nano 3d model with headers
Parts:
- SW25: footprint my_library:RotaryEncoder_Alps_EC11E-Switch_Vertical_H20mm -> autotome_library:RotaryEncoder_Alps_EC11E-Switch_Vertical_H20mm
- U1: footprint kbd:ProMicro -> autotome_library:NiceNano
Changed lines of the file:
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@@
 			)
 		)
-		(property "Footprint" "kbd:ProMicro"
+		(property "Footprint" "autotome_library:NiceNano"
 			(at 46.99 64.77 0)
 			(hide yes)
@@
 			)
 		)
-		(property "Footprint" "my_library:RotaryEncoder_Alps_EC11E-Switch_Vertical_H20mm"
+		(property "Footprint" "autotome_library:RotaryEncoder_Alps_EC11E-Switch_Vertical_H20mm"
 			(at 153.924 104.14 0)
 			(hide yes)

Commit message: move battery+ to correct pin on switch
Connections:
- net at SW31.1 (A): no longer BT1.1 (+)
- net at SW31.2 (B): now also BT1.1 (+)
Other:
- moved on the sheet: BT1
Changed lines of the file:
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@@
 	(wire
 		(pts
-			(xy 97.79 43.18) (xy 104.14 43.18)
-		)
-		(stroke
-			(width 0)
-			(type default)
-		)
-	)
-	(wire
-		(pts
 			(xy 86.36 123.19) (xy 104.14 123.19)
 		)
@@
 	(wire
 		(pts
+			(xy 95.25 27.94) (xy 95.25 33.02)
+		)
+		(stroke
+			(width 0)
+			(type default)
+		)
+	)
+	(wire
+		(pts
 			(xy 50.8 102.87) (xy 68.58 102.87)
 		)
@@
 	(global_label "B-"
 		(shape input)
-		(at 111.76 43.18 0)
+		(at 102.87 27.94 0)
 		(fields_autoplaced yes)
 		(effects
@@
 		)
 		(property "Intersheetrefs" "${INTERSHEET_REFS}"
-			(at 117.5876 43.18 0)
+			(at 108.6976 27.94 0)
 			(hide yes)
 			(show_name no)
@@
 	(symbol
 		(lib_id "Device:Battery_Cell")
-		(at 109.22 43.18 90)
+		(at 100.33 27.94 90)
 		(unit 1)
 		(body_style 1)
@@
 		(fields_autoplaced yes)
 		(property "Reference" "BT1"
-			(at 107.3785 35.56 90)
+			(at 98.4885 20.32 90)
 			(show_name no)
 			(do_not_autoplace no)
@@
 		)
 		(property "Value" "Battery_Cell"
-			(at 107.3785 38.1 90)
+			(at 98.4885 22.86 90)
 			(show_name no)
 			(do_not_autoplace no)
@@
 		)
 		(property "Footprint" "Connector_JST:JST_XH_B2B-XH-A_1x02_P2.50mm_Vertical"
-			(at 107.696 43.18 90)
+			(at 98.806 27.94 90)
 			(hide yes)
 			(show_name no)
@@
 		)
 		(property "Datasheet" ""
-			(at 107.696 43.18 90)
+			(at 98.806 27.94 90)
 			(hide yes)
 			(show_name no)
@@
 		)
 		(property "Description" "Single-cell battery"
-			(at 109.22 43.18 0)
+			(at 100.33 27.94 0)
 			(hide yes)
 			(show_name no)
@@
 		)
 		(property "Sim.Device" "V"
-			(at 109.22 43.18 0)
+			(at 100.33 27.94 0)
 			(hide yes)
 			(show_name no)
@@
 		)
 		(property "Sim.Type" "DC"
-			(at 109.22 43.18 0)
+			(at 100.33 27.94 0)
 			(hide yes)
 			(show_name no)
@@
 		)
 		(property "Sim.Pins" "1=+ 2=-"
-			(at 109.22 43.18 0)
+			(at 100.33 27.94 0)
 			(hide yes)
 			(show_name no)

Commit message: fix button number order in schematic, update pcb
Parts:
- renumbered D27 to D25, D28 to D26, D29 to D27, D30 to D28, D25 to RE1D1, SW25 to RE1SW1, SW31 to SLSW1, SW27 to SW25, SW28 to SW26, SW29 to SW27, SW30 to SW28
Changed lines of the file:
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@@
 		(in_pos_files yes)
 		(dnp no)
-		(property "Reference" "SW27"
+		(property "Reference" "SW25"
 			(at 60.96 124.46 0)
 			(show_name no)
@@
 			(project "autotome"
 				(path "/7a8f7727-35b5-4a31-8719-22ef542e3f8e"
-					(reference "SW27")
+					(reference "SW25")
 					(unit 1)
 				)
@@
 		(in_pos_files yes)
 		(dnp no)
-		(property "Reference" "SW31"
+		(property "Reference" "SLSW1"
 			(at 85.09 36.576 90)
 			(show_name no)
@@
 			(project "autotome"
 				(path "/7a8f7727-35b5-4a31-8719-22ef542e3f8e"
-					(reference "SW31")
+					(reference "SLSW1")
 					(unit 1)
 				)
@@
 		(in_pos_files yes)
 		(dnp no)
-		(property "Reference" "D28"
+		(property "Reference" "D26"
 			(at 85.09 129.54 90)
 			(show_name no)
@@
 			(project "autotome"
 				(path "/7a8f7727-35b5-4a31-8719-22ef542e3f8e"
-					(reference "D28")
+					(reference "D26")
 					(unit 1)
 				)
@@
 		(in_pos_files yes)
 		(dnp no)
-		(property "Reference" "D27"
+		(property "Reference" "D25"
 			(at 67.31 129.54 90)
 			(show_name no)
@@
 			(project "autotome"
 				(path "/7a8f7727-35b5-4a31-8719-22ef542e3f8e"
-					(reference "D27")
+					(reference "D25")
 					(unit 1)
 				)
@@
 		(in_pos_files yes)
 		(dnp no)
-		(property "Reference" "SW30"
+		(property "Reference" "SW28"
 			(at 114.3 124.46 0)
 			(show_name no)
@@
 			(project "autotome"
 				(path "/7a8f7727-35b5-4a31-8719-22ef542e3f8e"
-					(reference "SW30")
+					(reference "SW28")
 					(unit 1)
 				)
@@
 		(dnp no)
 		(fields_autoplaced yes)
-		(property "Reference" "SW25"
+		(property "Reference" "RE1SW1"
 			(at 156.21 106.6799 90)
 			(show_name no)
@@
 			(project "autotome"
 				(path "/7a8f7727-35b5-4a31-8719-22ef542e3f8e"
-					(reference "SW25")
+					(reference "RE1SW1")
 					(unit 1)
 				)
@@
 		(in_pos_files yes)
 		(dnp no)
-		(property "Reference" "D29"
+		(property "Reference" "D27"
 			(at 102.87 129.54 90)
 			(show_name no)
@@
 			(project "autotome"
 				(path "/7a8f7727-35b5-4a31-8719-22ef542e3f8e"
-					(reference "D29")
+					(reference "D27")
 					(unit 1)
 				)
@@
 		(in_pos_files yes)
 		(dnp no)
-		(property "Reference" "D30"
+		(property "Reference" "D28"
 			(at 120.65 129.54 90)
 			(show_name no)
@@
 			(project "autotome"
 				(path "/7a8f7727-35b5-4a31-8719-22ef542e3f8e"
-					(reference "D30")
+					(reference "D28")
 					(unit 1)
 				)
@@
 		(in_pos_files yes)
 		(dnp no)
-		(property "Reference" "SW29"
+		(property "Reference" "SW27"
 			(at 96.52 124.46 0)
 			(show_name no)
@@
 			(project "autotome"
 				(path "/7a8f7727-35b5-4a31-8719-22ef542e3f8e"
-					(reference "SW29")
+					(reference "SW27")
 					(unit 1)
 				)
@@
 		(in_pos_files yes)
 		(dnp no)
-		(property "Reference" "SW28"
+		(property "Reference" "SW26"
 			(at 78.74 124.46 0)
 			(show_name no)
@@
 			(project "autotome"
 				(path "/7a8f7727-35b5-4a31-8719-22ef542e3f8e"
-					(reference "SW28")
+					(reference "SW26")
 					(unit 1)
 				)
@@
 		(in_pos_files yes)
 		(dnp no)
-		(property "Reference" "D25"
+		(property "Reference" "RE1D1"
 			(at 149.606 120.65 90)
 			(show_name no)
@@
 			(project "autotome"
 				(path "/7a8f7727-35b5-4a31-8719-22ef542e3f8e"
-					(reference "D25")
+					(reference "RE1D1")
 					(unit 1)
 				)
