File: pcb/autotome.kicad_pcb (KiCad board)
At the start: 2 copper layers, 137 x 112.3 mm, 130 parts, among them SW1 SW_PUSH, SW10 SW_PUSH, SW11 SW_PUSH, SW12 SW_PUSH, SW13 SW_PUSH, SW14 SW_PUSH, SW15 SW_PUSH, SW16 SW_PUSH, SW17 SW_PUSH, SW18 SW_PUSH, SW19 SW_PUSH, SW2 SW_PUSH, SW20 SW_PUSH, SW21 SW_PUSH, SW22 SW_PUSH, SW23 SW_PUSH, SW24 SW_PUSH, SW25 SW_PUSH, SW26 SW_PUSH, SW27 SW_PUSH, SW28 SW_PUSH, SW29 SW_PUSH, SW3 SW_PUSH, SW30 SW_PUSH, SW31 SW_PUSH, SW32 SW_PUSH, SW33 SW_PUSH, SW34 SW_PUSH, SW35 SW_PUSH, SW36 SW_PUSH, SW37 SW_PUSH, SW38 SW_PUSH, SW39 SW_PUSH, SW4 SW_PUSH, SW40 SW_PUSH, SW41 SW_PUSH, SW42 SW_PUSH, SW43 SW_PUSH, SW44 SW_PUSH, SW45 SW_PUSH, SW46 SW_PUSH, SW47 SW_PUSH, SW48 SW_PUSH, SW49 SW_PUSH, SW5 SW_PUSH, SW50 SW_PUSH, SW51 SW_PUSH, SW52 SW_PUSH, SW53 SW_PUSH, SW54 SW_PUSH, SW55 SW_PUSH, SW56 SW_PUSH, SW6 SW_PUSH, SW7 SW_PUSH, SW8 SW_PUSH, SW9 SW_PUSH, U1 ProMicro, U2 ProMicro

Commit message: fix screw holes, add new ones for breakaway
Parts:
- removed the REF** at (83.2, 116.3)
- removed the REF** at (114.0, 77.2)
- removed the REF** at (37.8, 81.3)
- removed the REF** at (133.2, 119.8)
- added REF**: MountingHole_2.7mm_M2.5, MountingHole:MountingHole_2.7mm_M2.5, F.Cu at (114.6, 59.5)
- added REF**: MountingHole_2.7mm_M2.5, MountingHole:MountingHole_2.7mm_M2.5, F.Cu at (37.8, 81.0)
- added REF**: MountingHole_2.7mm_M2.5, MountingHole:MountingHole_2.7mm_M2.5, F.Cu at (37.8, 61.9)
- added REF**: MountingHole_2.7mm_M2.5, MountingHole:MountingHole_2.7mm_M2.5, F.Cu at (83.2, 115.8)
- added REF**: MountingHole_2.7mm_M2.5, MountingHole:MountingHole_2.7mm_M2.5, F.Cu at (113.4, 76.2)
- added REF**: MountingHole_2.7mm_M2.5, MountingHole:MountingHole_2.7mm_M2.5, F.Cu at (132.7, 119.7)
- moved D32 19.1 mm to (247.3, 52.4)
- moved D38 19.1 mm to (247.3, 71.4)
- moved D44 19.1 mm to (247.3, 90.5)
- moved D50 19.1 mm to (247.3, 109.5)
- moved D30 19.1 mm to (209.2, 52.4)
- moved D34 19.1 mm to (285.4, 57.2)
- moved D36 19.1 mm to (209.2, 71.4)
- moved D40 19.1 mm to (285.4, 76.2)
- moved D42 19.1 mm to (209.2, 90.5)
- moved D46 19.1 mm to (285.4, 95.3)
- moved D48 19.1 mm to (209.2, 109.5)
- moved D52 19.1 mm to (285.4, 114.3)
- moved D55 19.1 mm to (218.8, 132.4)
- moved D29 19.0 mm to (190.2, 54.8)
- moved D31 19.0 mm to (228.3, 50.0)
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
Commit message: complete right half edge cut
Parts:
- added REF**: MouseBite-Slot_2.0x2.0mm_inset_D0.5mm_P0.85mm_4h_Trace, Panelization:MouseBite-Slot_2.0x2.0mm_inset_D0.5mm_P0.85mm_4h_Trace, F.Cu at (283.4, 66.7)
- added REF**: MountingHole_2.7mm_M2.5, MountingHole:MountingHole_2.7mm_M2.5, F.Cu at (197.5, 80.0)
- added REF**: MountingHole_2.7mm_M2.5, MountingHole:MountingHole_2.7mm_M2.5, F.Cu at (273.2, 84.7)
- added REF**: MouseBite-Slot_2.0x2.0mm_inset_D0.5mm_P0.85mm_4h_Trace, Panelization:MouseBite-Slot_2.0x2.0mm_inset_D0.5mm_P0.85mm_4h_Trace, F.Cu at (244.6, 61.9)
- added REF**: MountingHole_2.7mm_M2.5, MountingHole:MountingHole_2.7mm_M2.5, F.Cu at (273.2, 65.7)
- added REF**: MouseBite-Slot_2.0x2.0mm_inset_D0.5mm_P0.85mm_4h_Trace, Panelization:MouseBite-Slot_2.0x2.0mm_inset_D0.5mm_P0.85mm_4h_Trace, F.Cu at (187.4, 64.3)
- added REF**: MountingHole_2.7mm_M2.5, MountingHole:MountingHole_2.7mm_M2.5, F.Cu at (196.4, 63.3)
- added REF**: MountingHole_2.7mm_M2.5, MountingHole:MountingHole_2.7mm_M2.5, F.Cu at (178.2, 123.5)
- added REF**: MouseBite-Slot_2.0x2.0mm_inset_D0.5mm_P0.85mm_4h_Trace, Panelization:MouseBite-Slot_2.0x2.0mm_inset_D0.5mm_P0.85mm_4h_Trace, F.Cu at (225.6, 59.5)
- added REF**: MountingHole_2.7mm_M2.5, MountingHole:MountingHole_2.7mm_M2.5, F.Cu at (227.8, 119.6)
- U2: moved to B.Cu
- moved U2 270.9 mm to (165.1, 81.2), turned to 180 degrees
- moved RE1D2 242.2 mm to (167.2, 127.5), turned to 180 degrees
- moved BT2 237.5 mm to (159.1, 101.8)
- moved SLSW2 225.0 mm to (171.7, 104.3), turned to 90 degrees
- moved RE1SW2 210.3 mm to (165.8, 110.0), turned to -90 degrees
- moved SLSW1 14.0 mm to (127.6, 104.3)
- moved D53 13.1 mm to (168.5, 146.8)
- moved D39 12.8 mm to (254.1, 80.0)
- moved D45 12.8 mm to (254.1, 99.0)
- moved D56 12.8 mm to (230.0, 136.2)
- moved SW49 12.8 mm to (225.5, 106.2)
- moved D31 12.8 mm to (216.0, 53.8)
- moved D33 12.8 mm to (254.1, 60.9)
- moved SW31 12.8 mm to (225.5, 49.0)
- moved D29 12.8 mm to (177.9, 58.5)
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Other:
- board size 137 x 112.3 mm -> 286.8 x 112.3 mm

Commit message: another route
Parts:
- U2: moved to F.Cu
- moved D33 3.00 mm to (254.1, 57.9)
- moved BT2 2.50 mm to (161.6, 101.8), turned to 180 degrees
- turned U2 to 0 degrees
Connections:
- U1 pad 13: col 5 -> col 0
- U1 pad 14: col 4 -> col 1
- U1 pad 15: col 3 -> col 2
- U1 pad 16: col 2 -> col 3
- U1 pad 17: col 1 -> col 4
- U1 pad 18: col 0 -> col 5
Routing:
- net col 4r: track 0.00 -> 251.1 mm
- net col 1: track 0.00 -> 248.8 mm
- net col 0: track 0.00 -> 248.4 mm, vias 0 -> 2
- net col 5r: track 0.00 -> 243.6 mm
- net col 3r: track 0.00 -> 235.2 mm
- net col 2: track 0.00 -> 217.4 mm
- net col 2r: track 0.00 -> 203.6 mm
- net col 3: track 0.00 -> 202.3 mm
- net col 1r: track 0.00 -> 198.1 mm
- net col 4: track 0.00 -> 191.4 mm
- net row 3r: track 0.00 -> 165.7 mm
- net row 3: track 0.00 -> 164.8 mm
- net col 0r: track 0.00 -> 156.2 mm
- net col 5: track 0.00 -> 153.0 mm
- net row 0r: track 0.00 -> 142.9 mm
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
Commit message: copper pour
Routing:
- added copper zone on B.Cu, net (none)
- added copper zone on F.Cu, net (none)
Changed lines of the file:
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@@
 		(net "Net-(D56-A)")
+	)
+	(zone
+		(layers "F.Cu" "B.Cu")
+		(hatch edge 0.5)
+		(connect_pads
+			(clearance 0.5)
+		)
+		(min_thickness 0.25)
+		(fill yes
+			(thermal_gap 0.5)
+			(thermal_bridge_width 0.5)
+			(island_removal_mode 1)
+		)
+		(polygon
+			(pts
+				(xy -5.150232 28.485744) (xy 302.939768 28.485744) (xy 302.939768 163.255744) (xy -8.080232 163.255744)
+			)
+		)
 	)
 	(embedded_fonts no)
